Commit message: modification

File: ur3_gazebo/urdf/ur3e.xacro (robot description, xacro)
@@ -65,5 +65,5 @@
     <parent link="world"/>
     <child link="base_link"/>
-    <origin xyz="0 0 0.1" rpy="0 0 0"/>
+    <origin xyz="0 0 0.105" rpy="0 0 0"/>
   </joint>
 </robot>

File: ur3_gazebo/urdf/ur_gripper_hande_ft300s.xacro (robot description, xacro)
@@ -65,5 +65,5 @@
     <parent link="world"/>
     <child link="base_link"/>
-    <origin xyz="0 0 0.1" rpy="0 0 0"/>
+    <origin xyz="0 0 0.105" rpy="0 0 0"/>
   </joint>
   <!-- Tf sensor -->
