Commit message: add

File: ur3_gazebo/urdf/ur_gripper_hande.xacro (robot description, xacro)
@@ -70,4 +70,30 @@
   <xacro:arg name="grasp_plugin" default="false" />
   <xacro:include filename="$(find ur3_gazebo)/urdf/robotiq_hande_gripper.urdf.xacro" />
+  <!-- camera mount -->
+  <link name="camera_mount">
+    <inertial>
+        <origin xyz="0 0 0" rpy="0 0 0"/>
+        <mass value="0.65"/>
+        <inertia ixx="0.000661171875" ixy="0" ixz="0" iyy="0.000661171875" iyz="0" izz="0.00117" />
+    </inertial>
+    <visual>
+        <origin xyz="0.0158 -0.033 0.01" rpy="${-pi/2} 0 ${pi}" />
+        <geometry>
+            <mesh filename="package://ur3_gazebo/mesh/mount_1.stl" scale="0.001 0.001 0.001"/>
+        </geometry>
+        <material name="black"/>
+    </visual>
+    <collision>
+        <origin xyz="0.0158 -0.033 0.01" rpy="${-pi/2} 0 ${pi}" />
+        <geometry>
+            <mesh filename="package://ur3_gazebo/mesh/mount_1.stl" scale="0.001 0.001 0.001"/>
+        </geometry>
+    </collision>
+  </link>
+  <joint name="camera_joint" type="fixed">
+    <origin xyz="0 0 0.00" rpy="0 0 0" />
+    <parent link="tool0"/>
+    <child link="camera_mount"/>
+  </joint>
   <!-- Robotiq Coupler -->
   <!--  + Height added by the coupler: 8mm -->

Commit message: fix

File: ur3_gazebo/urdf/ur_gripper_hande.xacro (robot description, xacro)
@@ -82,5 +82,4 @@
             <mesh filename="package://ur3_gazebo/mesh/mount_1.stl" scale="0.001 0.001 0.001"/>
         </geometry>
-        <material name="black"/>
     </visual>
     <collision>
@@ -104,5 +103,4 @@
         <mesh filename="package://robotiq_description/meshes/robotiq_85_coupler.stl" />
       </geometry>
-      <material name="flat_black"/>
     </visual>
     <collision>
@@ -126,5 +124,4 @@
     <mu1>0.9</mu1>
     <mu2>0.9</mu2>
-    <material>Gazebo/FlatBlack</material>
   </gazebo>
   <!-- Equivalent to the OpenRAVE manipulator denso_robotiq_hande_gripper -->

Commit message: add cameracalibration and fix

File: ur3_gazebo/urdf/ur_gripper_hande.xacro (robot description, xacro)
@@ -65,5 +65,5 @@
     <parent link="world"/>
     <child link="base_link"/>
-    <origin xyz="0 0 0.105" rpy="0 0 0"/>
+    <origin xyz="0 0 0.0" rpy="0 0 0"/>
   </joint>
   <!-- Gripper -->
